Commit message: add meshes

File: robots/kobuki_custom_velodyne-vlp16.urdf.xacro (robot description, xacro)
@@ -12,20 +12,21 @@
   <kobuki/>
   <VLP-16 parent="base_link" gpu="$(arg ray_gpu)" >
-    <origin xyz="0 0 ${0.0782 + 0.127}" rpy="0 0 0" />
+    <origin xyz="0 0 ${0.088 + 0.126}" rpy="0 0 0" />
   </VLP-16>
   <joint name="custom_stack_joint" type="fixed">
     <parent link="base_link"/>
     <child link="custom_stack"/>
-    <origin xyz="0 0 ${0.0782 + 0.127/2}" rpy="0 0 0"/>
+    <origin xyz="0 0 ${0.088 + 0.126/2}" rpy="0 0 0"/>
   </joint>
   <link name="custom_stack">
     <visual>
+      <origin xyz="0 0 -${0.126/2}" rpy="0 0 -1.570796"/>
       <geometry>
-        <box size="0.12 0.145 0.127"/>
+        <mesh filename="package://lidar_turtlebot/meshes/custom_stack.stl" scale="0.001 0.001 0.001"/>
       </geometry>
     </visual>
     <collsion>
       <geometry>
-        <box size="0.12 0.145 0.127"/>
+        <box size="0.12 0.146 0.126"/>
       </geometry>
     </collsion>

Commit message: Add imu and gps to urdf

File: robots/kobuki_custom_velodyne-vlp16.urdf.xacro (robot description, xacro)
@@ -32,3 +32,42 @@
     </collsion>
   </link>
+  <joint name="gps_joint" type="fixed">
+    <parent link="base_link"/>
+    <child link="gps"/>
+    <origin xyz="0 0.113 ${0.088 + 0.092 + 0.0195/2}" rpy="0 0 0"/>
+  </joint>
+  <link name="gps">
+    <visual>
+      <origin xyz="0 0 -${0.0195/2}" rpy="0 0 3.14159"/>
+      <geometry>
+        <mesh filename="package://lidar_turtlebot/meshes/GPS_garmin.stl" scale="0.001 0.001 0.001"/>
+      </geometry>
+    </visual>
+    <collsion>
+      <geometry>
+        <cylinder radius="0.03" length="0.01"/>
+      </geometry>
+    </collsion>
+  </link>
+  <joint name="imu_joint" type="fixed">
+    <parent link="base_link"/>
+    <child link="imu"/>
+    <origin xyz="0 0 ${0.088 + 0.1121}" rpy="0 0 0"/>
+  </joint>
+  <link name="imu">
+    <visual>
+      <origin xyz="0 0  -${0.0016/2 + 0.0005}" rpy="0 0 0"/>
+<!--      <origin xyz="${0.03175/2 + 0.0239 + 0.0015} ${0.03175/2 + 0.015 + 0.0015}  -${0.0016/2 + 0.0005}" rpy="0 0 0"/>-->
+      <geometry>
+        <box size="0.03175 0.03175 0.0016"/>
+        <!-- <mesh filename="package://lidar_turtlebot/meshes/sparkfun-9dof-razor-imu.stl" scale="0.001 0.001 0.001"/>-->
+      </geometry>
+    </visual>
+    <collsion>
+      <origin xyz="0 0  -${0.0016/2 + 0.0005}" rpy="0 0 0"/>
+      <geometry>
+        <box size="0.03175 0.03175 0.0016"/>
+      </geometry>
+    </collsion>
+  </link>
 </robot>

Commit message: change link name of imu

File: robots/kobuki_custom_velodyne-vlp16.urdf.xacro (robot description, xacro)
@@ -52,8 +52,8 @@
   <joint name="imu_joint" type="fixed">
     <parent link="base_link"/>
-    <child link="imu"/>
+    <child link="base_imu_link"/>
     <origin xyz="0 0 ${0.088 + 0.1121}" rpy="0 0 0"/>
   </joint>
-  <link name="imu">
+  <link name="base_imu_link">
     <visual>
       <origin xyz="0 0  -${0.0016/2 + 0.0005}" rpy="0 0 0"/>
