Commit message: fix file path

File: lidar_turtlebot_description/robots/kobuki_custom_velodyne-vlp16.urdf.xacro (robot description, xacro)
@@ -23,5 +23,5 @@
       <origin xyz="0 0 -${0.126/2}" rpy="0 0 -1.570796"/>
       <geometry>
-        <mesh filename="package://lidar_turtlebot/meshes/custom_stack.stl" scale="0.001 0.001 0.001"/>
+        <mesh filename="package://lidar_turtlebot_description/meshes/custom_stack.stl" scale="0.001 0.001 0.001"/>
       </geometry>
     </visual>
@@ -41,5 +41,5 @@
       <origin xyz="0 0 -${0.0195/2}" rpy="0 0 3.14159"/>
       <geometry>
-        <mesh filename="package://lidar_turtlebot/meshes/GPS_garmin.stl" scale="0.001 0.001 0.001"/>
+        <mesh filename="package://lidar_turtlebot_description/meshes/GPS_garmin.stl" scale="0.001 0.001 0.001"/>
       </geometry>
     </visual>
@@ -61,5 +61,5 @@
       <geometry>
         <box size="0.03175 0.03175 0.0016"/>
-        <!-- <mesh filename="package://lidar_turtlebot/meshes/sparkfun-9dof-razor-imu.stl" scale="0.001 0.001 0.001"/>-->
+        <!-- <mesh filename="package://lidar_turtlebot_description/meshes/sparkfun-9dof-razor-imu.stl" scale="0.001 0.001 0.001"/>-->
       </geometry>
     </visual>
