Commit message: launch files for load model and pointcloud to navigation_laserscan

File: lidar_turtlebot_description/robots/kobuki_custom_rplidar-a2.urdf.xacro (robot description, xacro)
@@ -17,13 +17,20 @@
   <link name="rplidar">
     <visual>
-      <origin xyz="-0.007 -0.075 -0.038" rpy="${pi/2} 0 ${pi}"/>
+      <!--<origin xyz="-0.007 -0.075 -0.038" rpy="${pi/2} 0 ${pi}"/>-->
+      <origin xyz="-0.006 -0.075 ${-0.008 - 0.0308}" rpy="${pi/2} 0 ${pi}"/>
       <geometry>
-        <mesh filename="package://lidar_turtlebot/meshes/rplidar-a2m4-r1.stl"/>
+        <mesh filename="package://lidar_turtlebot_description/meshes/rplidar-a2m4-r1.stl"/>
+      </geometry>
+    </visual>
+    <visual>
+      <origin xyz="0 0 ${-0.0308 -0.0069}" rpy="0 0 0"/>
+      <geometry>
+        <mesh filename="package://lidar_turtlebot_description/meshes/RPLidar_holder.stl"/>
       </geometry>
     </visual>
     <collsion>
-      <origin xyz="0 0 ${0.0408 / 2 -0.0306}" rpy="0 0 0"/>
+      <origin xyz="0 0 ${(0.0408 + 0.0069)/ 2 -0.0306}" rpy="0 0 0"/>
       <geometry>
-        <cylinder radius="${0.0757 / 2}" length="0.0408"/>
+        <cylinder radius="${0.0757 / 2}" length="${0.0408 + 0.0069}"/>
       </geometry>
     </collsion>
@@ -38,5 +45,5 @@
       <origin xyz="0 0 -${0.126/2}" rpy="0 0 -1.570796"/>
       <geometry>
-        <mesh filename="package://lidar_turtlebot/meshes/custom_stack.stl" scale="0.001 0.001 0.001"/>
+        <mesh filename="package://lidar_turtlebot_description/meshes/custom_stack.stl" scale="0.001 0.001 0.001"/>
       </geometry>
     </visual>
@@ -56,5 +63,5 @@
       <origin xyz="0 0 -${0.0195/2}" rpy="0 0 3.14159"/>
       <geometry>
-        <mesh filename="package://lidar_turtlebot/meshes/GPS_garmin.stl" scale="0.001 0.001 0.001"/>
+        <mesh filename="package://lidar_turtlebot_description/meshes/GPS_garmin.stl" scale="0.001 0.001 0.001"/>
       </geometry>
     </visual>
@@ -76,5 +83,5 @@
       <geometry>
         <box size="0.03175 0.03175 0.0016"/>
-        <!-- <mesh filename="package://lidar_turtlebot/meshes/sparkfun-9dof-razor-imu.stl" scale="0.001 0.001 0.001"/>-->
+        <!-- <mesh filename="package://lidar_turtlebot_description/meshes/sparkfun-9dof-razor-imu.stl" scale="0.001 0.001 0.001"/>-->
       </geometry>
     </visual>

File: lidar_turtlebot_description/robots/kobuki_custom_velodyne-vlp16.urdf.xacro (robot description, xacro)
@@ -6,5 +6,5 @@
 -->
 <robot name="turtlebot" xmlns:xacro="http://ros.org/wiki/xacro">
-  <xacro:arg name="ray_gpu" default="true"/>
+  <xacro:arg name="ray_gpu" default="false"/>
   <xacro:include filename="$(find turtlebot_description)/urdf/turtlebot_common_library.urdf.xacro" />
   <xacro:include filename="$(find kobuki_description)/urdf/kobuki.urdf.xacro" />
